File: CarbonAwareCircuit.kicad_sch (KiCad schematic)
At the start: 3 parts, among them J1 USB_C_Receptacle_PowerOnly_6P, U1 LD1117V33, U2 ESP32-C3

Commit message: more eeschema updates
Connections:
- net at U2.33 (GND): now also J1.A12 (GND), J1.B12 (GND), J1.SH (SHIELD), U1.1 (GND)
Other:
- moved on the sheet: U2
Changed lines of the file:
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@@
 		(rev "1.0")
+	)
+	(junction
+		(at 31.75 52.07)
+		(diameter 0)
+		(color 0 0 0 0)
 	)
 	(wire
@@
 	(wire
 		(pts
+			(xy 31.75 72.39) (xy 49.53 72.39)
+		)
+		(stroke
+			(width 0)
+			(type default)
+		)
+	)
+	(wire
+		(pts
 			(xy 46.99 26.67) (xy 67.31 26.67)
+		)
+		(stroke
+			(width 0)
+			(type default)
+		)
+	)
+	(wire
+		(pts
+			(xy 24.13 52.07) (xy 31.75 52.07)
 		)
 		(stroke
@@
 		)
 	)
+	(wire
+		(pts
+			(xy 31.75 52.07) (xy 31.75 72.39)
+		)
+		(stroke
+			(width 0)
+			(type default)
+		)
+	)
 	(symbol
 		(lib_id "MCU_Espressif:ESP32-C3")
-		(at 74.93 72.39 0)
+		(at 74.93 72.39 270)
 		(unit 1)
 		(body_style 1)
@@
 		(fields_autoplaced yes)
 		(property "Reference" "U2"
-			(at 77.0733 97.79 0)
+			(at 45.72 65.9698 90)
 			(show_name no)
 			(do_not_autoplace no)
@@
 					(size 1.27 1.27)
 				)
-				(justify left)
 			)
 		)
 		(property "Value" "ESP32-C3"
-			(at 77.0733 100.33 0)
+			(at 45.72 68.5098 90)
 			(show_name no)
 			(do_not_autoplace no)
@@
 					(size 1.27 1.27)
 				)
-				(justify left)
 			)
 		)
 		(property "Footprint" "Package_DFN_QFN:QFN-32-1EP_5x5mm_P0.5mm_EP3.7x3.7mm"
-			(at 75.438 72.39 0)
+			(at 74.93 72.898 0)
 			(hide yes)
 			(show_name no)
@@
 		)
 		(property "Datasheet" "https://www.espressif.com/sites/default/files/documentation/esp32-c3_datasheet_en.pdf"
-			(at 75.438 72.39 0)
+			(at 74.93 72.898 0)
 			(hide yes)
 			(show_name no)
@@
 		)
 		(property "Description" "RF Module, ESP32 SoC, RISC-V, WiFi 802.11b/n/g, Bluetooth LE 5, QFN32"
-			(at 75.438 72.39 0)
+			(at 74.93 72.898 0)
 			(hide yes)
 			(show_name no)

Commit message: more circuit tweaks
Parts:
- removed J1: USB_C_Receptacle_PowerOnly_6P, symbol Connector:USB_C_Receptacle_PowerOnly_6P
- added D1: LED, symbol Device:LED
- added J1: USB_C_Receptacle_USB2.0_14P, symbol Connector:USB_C_Receptacle_USB2.0_14P
- added R1: R_Small, symbol Device:R_Small
Connections:
- net at U2.11 (VDD3P3_RTC): now also U1.2 (VO), U2.17 (VDD3P3_CPU), U2.18 (VDD_SPI), U2.2 (VDD3P3), U2.3 (VDD3P3), U2.31 (VDDA), U2.32 (VDDA)
- net at U1.1 (GND), U2.33 (GND): now also D1.1 (K), J1.A1 (GND), J1.A12 (GND), J1.B1 (GND), J1.B12 (GND), J1.SH (SHIELD)
- net at U2.6 (GPIO2): now also D1.2 (A)
- net at U1.3 (VI): now also J1.A4 (VBUS), J1.A9 (VBUS), J1.B4 (VBUS), J1.B9 (VBUS)
Other:
- moved on the sheet: U1, U2
