File: CarbonAwareCircuit.kicad_sch (KiCad schematic)
At the start: 11 parts, among them J1 USB_C_Receptacle_USB2.0_14P, SW1 SW_Push_Dual_x2, SW2 SW_Push_Dual_x2, U1 LD1117V33, U2 ESP32-C3-WROOM-02

Commit message: moved things around
Parts:
- D1: footprint (none) -> LED_THT:LED_D2.0mm_W4.8mm_H2.5mm_FlatTop
- J1: footprint (none) -> Connector_USB:USB_C_Receptacle_GCT_USB4125-xx-x_6P_TopMnt_Horizontal
- R1: footprint (none) -> Resistor_THT:R_Axial_DIN0309_L9.0mm_D3.2mm_P25.40mm_Horizontal
- R2, R4, R5, R6: footprint (none) -> Resistor_THT:R_Axial_DIN0411_L9.9mm_D3.6mm_P5.08mm_Vertical
- SW1: footprint (none) -> Button_Switch_THT:SW_DIP_SPSTx05_Piano_CTS_Series194-5MSTN_W7.62mm_P2.54mm
- SW2: footprint (none) -> Button_Switch_THT:SW_DIP_SPSTx03_Piano_10.8x9.18mm_W7.62mm_P2.54mm
Connections:
- no-connect marks 4 -> 5
Other:
- moved on the sheet: R4
Changed lines of the file:
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@@
 	)
 	(junction
-		(at 73.66 74.93)
+		(at 73.66 35.56)
 		(diameter 0)
 		(color 0 0 0 0)
@@
 	)
 	(junction
+		(at 74.93 74.93)
+		(diameter 0)
+		(color 0 0 0 0)
+	)
+	(junction
 		(at 45.72 38.1)
 		(diameter 0)
@@
 	)
 	(junction
-		(at 116.84 100.33)
-		(diameter 0)
-		(color 0 0 0 0)
-	)
-	(junction
-		(at 73.66 35.56)
+		(at 116.84 102.87)
 		(diameter 0)
 		(color 0 0 0 0)
@@
 	)
 	(no_connect
+		(at 116.84 49.53)
+	)
+	(no_connect
 		(at 88.9 52.07)
 	)
@@
 	(wire
 		(pts
+			(xy 74.93 74.93) (xy 76.2 74.93)
+		)
+		(stroke
+			(width 0)
+			(type default)
+		)
+	)
+	(wire
+		(pts
 			(xy 114.3 30.48) (xy 73.66 30.48)
 		)
@@
 	(wire
 		(pts
-			(xy 73.66 102.87) (xy 73.66 74.93)
+			(xy 74.93 102.87) (xy 74.93 74.93)
 		)
 		(stroke
@@
 	(wire
 		(pts
-			(xy 73.66 35.56) (xy 73.66 74.93)
+			(xy 74.93 35.56) (xy 74.93 74.93)
 		)
 		(stroke
@@
 	(wire
 		(pts
-			(xy 132.08 100.33) (xy 132.08 85.09)
+			(xy 148.59 102.87) (xy 148.59 85.09)
+		)
+		(stroke
+			(width 0)
+			(type default)
+		)
+	)
+	(wire
+		(pts
+			(xy 121.92 102.87) (xy 148.59 102.87)
+		)
+		(stroke
+			(width 0)
+			(type default)
+		)
+	)
+	(wire
+		(pts
+			(xy 148.59 85.09) (xy 132.08 85.09)
+		)
+		(stroke
+			(width 0)
+			(type default)
+		)
+	)
+	(wire
+		(pts
+			(xy 132.08 80.01) (xy 132.08 85.09)
 		)
 		(stroke
@@
 	(wire
 		(pts
-			(xy 73.66 74.93) (xy 76.2 74.93)
+			(xy 116.84 97.79) (xy 116.84 102.87)
 		)
 		(stroke
@@
 	(wire
 		(pts
-			(xy 121.92 100.33) (xy 132.08 100.33)
+			(xy 74.93 35.56) (xy 73.66 35.56)
 		)
 		(stroke
@@
 	(wire
 		(pts
-			(xy 55.88 74.93) (xy 73.66 74.93)
+			(xy 55.88 74.93) (xy 74.93 74.93)
 		)
 		(stroke
@@
 	(wire
 		(pts
-			(xy 116.84 102.87) (xy 116.84 100.33)
-		)
-		(stroke
-			(width 0)
-			(type default)
-		)
-	)
-	(wire
-		(pts
 			(xy 124.46 41.91) (xy 124.46 38.1)
 		)
@@
 	(wire
 		(pts
-			(xy 116.84 100.33) (xy 116.84 97.79)
-		)
-		(stroke
-			(width 0)
-			(type default)
-		)
-	)
-	(wire
-		(pts
 			(xy 73.66 30.48) (xy 73.66 35.56)
 		)
@@
 	(wire
 		(pts
-			(xy 132.08 80.01) (xy 132.08 85.09)
-		)
-		(stroke
-			(width 0)
-			(type default)
-		)
-	)
-	(wire
-		(pts
 			(xy 132.08 30.48) (xy 132.08 40.64)
 		)
@@
 	(wire
 		(pts
-			(xy 105.41 102.87) (xy 73.66 102.87)
+			(xy 105.41 102.87) (xy 74.93 102.87)
 		)
 		(stroke
@@
 			)
 		)
-		(property "Footprint" ""
+		(property "Footprint" "Resistor_THT:R_Axial_DIN0411_L9.9mm_D3.6mm_P5.08mm_Vertical"
 			(at 116.84 49.53 0)
 			(hide yes)
@@
 			)
 		)
-		(property "Footprint" ""
+		(property "Footprint" "Button_Switch_THT:SW_DIP_SPSTx03_Piano_10.8x9.18mm_W7.62mm_P2.54mm"
 			(at 110.49 107.95 0)
 			(hide yes)
@@
 			)
 		)
-		(property "Footprint" ""
+		(property "Footprint" "Resistor_THT:R_Axial_DIN0411_L9.9mm_D3.6mm_P5.08mm_Vertical"
 			(at 52.07 33.02 0)
 			(hide yes)
@@
 			)
 		)
-		(property "Footprint" ""
+		(property "Footprint" "Connector_USB:USB_C_Receptacle_GCT_USB4125-xx-x_6P_TopMnt_Horizontal"
 			(at 34.29 38.1 0)
 			(hide yes)
@@
 			)
 		)
-		(property "Footprint" ""
+		(property "Footprint" "Resistor_THT:R_Axial_DIN0309_L9.0mm_D3.2mm_P25.40mm_Horizontal"
 			(at 52.07 27.94 0)
 			(hide yes)
@@
 			)
 		)
-		(property "Footprint" ""
+		(property "Footprint" "Resistor_THT:R_Axial_DIN0411_L9.9mm_D3.6mm_P5.08mm_Vertical"
 			(at 124.46 44.45 0)
 			(hide yes)
@@
 			)
 		)
-		(property "Footprint" ""
+		(property "Footprint" "Button_Switch_THT:SW_DIP_SPSTx05_Piano_CTS_Series194-5MSTN_W7.62mm_P2.54mm"
 			(at 109.22 36.83 0)
 			(hide yes)
@@
 	(symbol
 		(lib_id "Device:R_Small")
-		(at 119.38 100.33 90)
+		(at 119.38 102.87 90)
 		(unit 1)
 		(body_style 1)
@@
 		(dnp no)
 		(property "Reference" "R4"
-			(at 120.142 98.552 90)
+			(at 120.142 101.092 90)
 			(show_name no)
 			(do_not_autoplace no)
@@
 		)
 		(property "Value" "10kΩ"
-			(at 122.174 102.362 90)
+			(at 122.174 104.902 90)
 			(show_name no)
 			(do_not_autoplace no)
@@
 			)
 		)
-		(property "Footprint" ""
-			(at 119.38 100.33 0)
+		(property "Footprint" "Resistor_THT:R_Axial_DIN0411_L9.9mm_D3.6mm_P5.08mm_Vertical"
+			(at 119.38 102.87 0)
 			(hide yes)
 			(show_name no)
@@
 		)
 		(property "Datasheet" ""
-			(at 119.38 100.33 0)
+			(at 119.38 102.87 0)
 			(hide yes)
 			(show_name no)
@@
 		)
 		(property "Description" "Resistor, small symbol"
-			(at 119.38 100.33 0)
+			(at 119.38 102.87 0)
 			(hide yes)
 			(show_name no)
@@
 			)
 		)
-		(property "Footprint" ""
+		(property "Footprint" "LED_THT:LED_D2.0mm_W4.8mm_H2.5mm_FlatTop"
 			(at 124.46 34.29 0)
 			(hide yes)

Commit message: decided to restart :(
Parts:
- removed D1: LED, LED_THT:LED_D2.0mm_W4.8mm_H2.5mm_FlatTop, symbol Device:LED
- removed R1: 5.1kΩ, Resistor_THT:R_Axial_DIN0309_L9.0mm_D3.2mm_P25.40mm_Horizontal, symbol Device:R_Small
- removed R2: 5.1kΩ, Resistor_THT:R_Axial_DIN0411_L9.9mm_D3.6mm_P5.08mm_Vertical, symbol Device:R_Small
- removed R4, R6: 10kΩ, Resistor_THT:R_Axial_DIN0411_L9.9mm_D3.6mm_P5.08mm_Vertical, symbol Device:R_Small
- removed R5: 330Ω, Resistor_THT:R_Axial_DIN0411_L9.9mm_D3.6mm_P5.08mm_Vertical, symbol Device:R_Small
- removed SW1: SW_Push_Dual_x2, Button_Switch_THT:SW_DIP_SPSTx05_Piano_CTS_Series194-5MSTN_W7.62mm_P2.54mm, symbol Switch:SW_Push_Dual_x2
- removed SW2: SW_Push_Dual_x2, Button_Switch_THT:SW_DIP_SPSTx03_Piano_10.8x9.18mm_W7.62mm_P2.54mm, symbol Switch:SW_Push_Dual_x2
- removed U1: LD1117V33, Package_TO_SOT_THT:TO-220-3_Vertical, symbol Regulator_Linear:LD1117V33
- removed U2: ESP32-C3-WROOM-02, Package_DFN_QFN:QFN-32-1EP_5x5mm_P0.5mm_EP3.7x3.7mm, symbol MCU_Espressif:ESP32-C3
- added U2: ESP32-C3-WROOM-02, RF_Module:ESP32-C3-WROOM-02, symbol RF_Module:ESP32-C3-WROOM-02
Connections:
- net at J1.A1 (GND), J1.A12 (GND), J1.B1 (GND)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: no longer J1.SH (SHIELD)
- net at J1.A6 (D+): no longer J1.B6 (D+)
- net at J1.A7 (D-): no longer J1.B7 (D-)
- new net: U2.19 (GND), U2.9 (GND)
- no-connect marks 5 -> 0
Other:
- moved on the sheet: J1
