File: CarbonAwareCircuit.kicad_pcb (KiCad board)
At the start: 2 copper layers, 64 x 52.5 mm, 15 parts, among them J1 USB_C_Receptacle_USB2.0_14P, J2 USB_A, Q1 AO3401A, SW1 SW_Push, SW2 SW_Push, U1 LD1117V, U2 ESP32-C3-WROOM-02

Commit message: pcb changes...
Routing:
- net Net-(Q1-S): track 52.7 -> 54.2 mm, vias 3 -> 5
Other:
- board size 64 x 52.5 mm -> 64 x 61.5 mm
Changed lines of the file:
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@@
 	)
 	(gr_rect
-		(start 192 88)
+		(start 192 79)
 		(end 256 140.5)
 		(stroke
@@
 	)
 	(segment
-		(start 235 129)
-		(end 232.2 131.8)
-		(width 1)
-		(layer "F.Cu")
-		(net "Net-(Q1-S)")
-	)
-	(segment
 		(start 229.803398 135.02)
 		(end 231.9 135.02)
@@
 	)
 	(segment
+		(start 235 129)
+		(end 234 129)
+		(width 1)
+		(layer "F.Cu")
+		(net "Net-(Q1-S)")
+	)
+	(segment
 		(start 232.2 134.72)
 		(end 232.2 134.12)
@@
 	)
 	(segment
-		(start 232.2 131.8)
-		(end 232.2 134.12)
-		(width 1)
-		(layer "F.Cu")
-		(net "Net-(Q1-S)")
-	)
-	(segment
 		(start 222.5 117.5)
 		(end 222.5 115.3)
@@
 	)
 	(via
+		(at 232.2 134.12)
+		(size 0.6)
+		(drill 0.3)
+		(layers "F.Cu" "B.Cu")
+		(net "Net-(Q1-S)")
+	)
+	(via
+		(at 234 129)
+		(size 0.6)
+		(drill 0.3)
+		(layers "F.Cu" "B.Cu")
+		(net "Net-(Q1-S)")
+	)
+	(via
 		(at 233.5 121)
 		(size 1)
@@
 	)
 	(segment
+		(start 234 129)
+		(end 232.5 129)
+		(width 1)
+		(layer "B.Cu")
+		(net "Net-(Q1-S)")
+	)
+	(segment
 		(start 235 122.5)
 		(end 235 125.5)
@@
 	)
 	(segment
+		(start 232.5 129)
+		(end 232.5 133.82)
+		(width 1)
+		(layer "B.Cu")
+		(net "Net-(Q1-S)")
+	)
+	(segment
 		(start 235 122.5)
 		(end 233.5 121)
 		(width 1)
 		(layer "B.Cu")
+		(net "Net-(Q1-S)")
+	)
+	(segment
+		(start 232.5 133.82)
+		(end 232.2 134.12)
+		(width 1)
+		(layer "B.Cu")
